Commit message: Raise active pitch joint upper limit 90->110 deg
The measured prone pitch (+100 deg, confirmed reachable on real hardware) was
outside the previous +90 deg active limit, which would clamp the pose or fail
pose validation. Raise the pitch upper limit to +110 deg (~1.9199 rad); the
lower limit (-90 deg) is unchanged. Safety-limit change, kept as its own commit.

File: urdf/leg.xacro (robot description, xacro)
@@ -143,5 +143,7 @@
       <parent link="${prefix}_pitch_holder_link"/><child link="${prefix}_thigh_link"/>
       <axis xyz="0 0 1"/>
-      <limit lower="${radians(-90)}" upper="${radians(90)}" effort="17" velocity="20"/>
+      <!-- upper raised 90->110deg so the measured prone pitch (+100deg, reachable
+           on real hardware) is inside the active limit; lower stays -90deg. -->
+      <limit lower="${radians(-90)}" upper="${radians(110)}" effort="17" velocity="20"/>
     </joint>
     <!-- active #3 (knee motor): thigh -> knee crank -->

Commit message: Lower active pitch joint limit to -110 deg for right-leg prone
Right-leg prone pitch is -100deg (mirrored from the left legs' +100deg) and was
reached on real hardware (RF -100.4, RR -99.6). Widen the active pitch lower
limit radians(-90) -> radians(-110), symmetric with the +110 upper, so the
mirrored prone pose is inside the active range on both sides. Safety-limit change.

File: urdf/leg.xacro (robot description, xacro)
@@ -143,7 +143,8 @@
       <parent link="${prefix}_pitch_holder_link"/><child link="${prefix}_thigh_link"/>
       <axis xyz="0 0 1"/>
-      <!-- upper raised 90->110deg so the measured prone pitch (+100deg, reachable
-           on real hardware) is inside the active limit; lower stays -90deg. -->
-      <limit lower="${radians(-90)}" upper="${radians(110)}" effort="17" velocity="20"/>
+      <!-- Symmetric +/-110deg active range so the measured prone pitch fits on
+           both sides: left legs reach +100deg, right legs -100deg (mirrored;
+           both reached on real hardware: RF -100.4, RR -99.6). -->
+      <limit lower="${radians(-110)}" upper="${radians(110)}" effort="17" velocity="20"/>
     </joint>
     <!-- active #3 (knee motor): thigh -> knee crank -->

Commit message: Widen active pitch limit to +/-110 deg for prone (squash)
Squash-merge feature/prone-pitch-limit: raise the active pitch joint upper limit
90->110 deg and lower limit to -110 deg so the measured prone pitch fits within
the active range. Latest body mesh/inertia export on main is preserved.

File: urdf/leg.xacro (robot description, xacro)
@@ -143,5 +143,8 @@
       <parent link="${prefix}_pitch_holder_link"/><child link="${prefix}_thigh_link"/>
       <axis xyz="0 0 1"/>
-      <limit lower="${radians(-90)}" upper="${radians(90)}" effort="17" velocity="20"/>
+      <!-- Symmetric +/-110deg active range so the measured prone pitch fits on
+           both sides: left legs reach +100deg, right legs -100deg (mirrored;
+           both reached on real hardware: RF -100.4, RR -99.6). -->
+      <limit lower="${radians(-110)}" upper="${radians(110)}" effort="17" velocity="20"/>
     </joint>
     <!-- active #3 (knee motor): thigh -> knee crank -->
